File: sl-pi-aprs.sch (KiCad schematic (older format))
At the start: 33 parts, among them J1 Power, J10 PTT Disable, J2 RPi Header, J3 Radio, J4 Radio In, J5 Audio In, J6 Audio In, J7 Audio Out, J8 Audio Out, J9 GPS Header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

Commit message: Add ground planes and minor adjustments
Parts:
- J9: footprint sl-pi-aprs:PinHeader_1x05_P2.54mm_Vertical_gt-u7_breakout -> Connector_JST:JST_XH_B5B-XH-A_1x05_P2.50mm_Vertical
Changed lines of the file:
@@
 F 0 "J9" H 10330 1842 50  0000 L CNN
 F 1 "GPS Header" H 10330 1751 50  0000 L CNN
-F 2 "sl-pi-aprs:PinHeader_1x05_P2.54mm_Vertical_gt-u7_breakout" H 10250 1800 50  0001 C CNN
+F 2 "Connector_JST:JST_XH_B5B-XH-A_1x05_P2.50mm_Vertical" H 10250 1800 50  0001 C CNN
 F 3 "~" H 10250 1800 50  0001 C CNN
 	1    10250 1800
